File: controls.kicad_sch (KiCad schematic)
At the start: 21 parts, among them J10 CV2, J11 IN2, J12 IN 1x8h, J13 OUT1, J14 OUT2, J5 CV 1x9h, J6 OUT 1x3h, J8 CV1, J9 IN1

Commit message: Updated controls and added licence
Connections:
- net GND: now also RV1.1, RV2.1; no longer RV1.3, RV2.3
- net at RV6.1: now also J12.8 (Pin_8); no longer J12.6 (Pin_6)
- net at RV6.3: now also J12.6 (Pin_6); no longer J12.8 (Pin_8)
- net at J10.T, J5.8 (Pin_8): now also RV2.3; no longer RV2.1
- net at J5.2 (Pin_2), J8.T: now also RV1.3; no longer RV1.1
- net at RV5.1: now also J12.4 (Pin_4); no longer J12.2 (Pin_2)
- net at RV5.3: now also J12.2 (Pin_2); no longer J12.4 (Pin_4)
- net at RV3.3: now also J5.5 (Pin_5), RV4.3
- now unconnected: RV3.1, RV4.1
Other:
- moved on the sheet: RV1, RV2
Changed lines of the file:
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@@
 		(lib_id "Device:R_Potentiometer")
 		(at 132.08 107.95 0)
-		(unit 1)
-		(body_style 1)
-		(exclude_from_sim no)
-		(in_bom yes)
-		(on_board yes)
-		(in_pos_files yes)
-		(dnp no)
-		(fields_autoplaced yes)
+		(mirror x)
+		(unit 1)
+		(body_style 1)
+		(exclude_from_sim no)
+		(in_bom yes)
+		(on_board yes)
+		(in_pos_files yes)
+		(dnp no)
 		(property "Reference" "RV6"
-			(at 129.54 106.6799 0)
+			(at 129.54 109.2201 0)
 			(show_name no)
 			(do_not_autoplace no)
@@
 		)
 		(property "Value" "10K B"
-			(at 129.54 109.2199 0)
+			(at 129.54 106.6801 0)
 			(show_name no)
 			(do_not_autoplace no)
@@
 	(symbol
 		(lib_id "Device:R_Potentiometer")
-		(at 44.45 109.22 90)
-		(unit 1)
-		(body_style 1)
-		(exclude_from_sim no)
-		(in_bom yes)
-		(on_board yes)
-		(in_pos_files yes)
-		(dnp no)
-		(fields_autoplaced yes)
+		(at 44.45 109.22 270)
+		(mirror x)
+		(unit 1)
+		(body_style 1)
+		(exclude_from_sim no)
+		(in_bom yes)
+		(on_board yes)
+		(in_pos_files yes)
+		(dnp no)
 		(property "Reference" "RV2"
 			(at 44.45 113.03 90)
@@
 	(symbol
 		(lib_id "Device:R_Potentiometer")
-		(at 44.45 53.34 90)
-		(unit 1)
-		(body_style 1)
-		(exclude_from_sim no)
-		(in_bom yes)
-		(on_board yes)
-		(in_pos_files yes)
-		(dnp no)
-		(fields_autoplaced yes)
+		(at 44.45 53.34 270)
+		(mirror x)
+		(unit 1)
+		(body_style 1)
+		(exclude_from_sim no)
+		(in_bom yes)
+		(on_board yes)
+		(in_pos_files yes)
+		(dnp no)
 		(property "Reference" "RV1"
 			(at 44.45 57.15 90)
@@
 		(lib_id "Device:R_Potentiometer")
 		(at 132.08 69.85 0)
-		(unit 1)
-		(body_style 1)
-		(exclude_from_sim no)
-		(in_bom yes)
-		(on_board yes)
-		(in_pos_files yes)
-		(dnp no)
-		(fields_autoplaced yes)
+		(mirror x)
+		(unit 1)
+		(body_style 1)
+		(exclude_from_sim no)
+		(in_bom yes)
+		(on_board yes)
+		(in_pos_files yes)
+		(dnp no)
 		(property "Reference" "RV5"
-			(at 129.54 68.5799 0)
+			(at 129.54 71.1201 0)
 			(show_name no)
 			(do_not_autoplace no)
@@
 		)
 		(property "Value" "10K B"
-			(at 129.54 71.1199 0)
+			(at 129.54 68.5801 0)
 			(show_name no)
 			(do_not_autoplace no)
@@
 		(lib_id "Device:R_Potentiometer")
 		(at 24.13 71.12 0)
-		(mirror x)
 		(unit 1)
 		(body_style 1)
@@
 		(dnp no)
 		(property "Reference" "RV3"
-			(at 21.59 72.3901 0)
+			(at 21.59 69.8499 0)
 			(show_name no)
 			(do_not_autoplace no)
@@
 		)
 		(property "Value" "50K B"
-			(at 21.59 69.8501 0)
+			(at 21.59 72.3899 0)
 			(show_name no)
 			(do_not_autoplace no)
@@
 		(lib_id "Device:R_Potentiometer")
 		(at 24.13 91.44 0)
-		(unit 1)
-		(body_style 1)
-		(exclude_from_sim no)
-		(in_bom yes)
-		(on_board yes)
-		(in_pos_files yes)
-		(dnp no)
-		(fields_autoplaced yes)
+		(mirror x)
+		(unit 1)
+		(body_style 1)
+		(exclude_from_sim no)
+		(in_bom yes)
+		(on_board yes)
+		(in_pos_files yes)
+		(dnp no)
 		(property "Reference" "RV4"
-			(at 21.59 90.1699 0)
+			(at 21.59 92.7101 0)
 			(show_name no)
 			(do_not_autoplace no)
@@
 		)
 		(property "Value" "50K B"
-			(at 21.59 92.7099 0)
-			(show_name no)
-			(do_not_autoplace no)
+			(at 21.59 90.1701 0)
+			(show_name no)
+			(do_not_autoplace no)

Commit message: Updated versioning
Other:
- note added: "V 1.1"
Changed lines of the file:
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@@
+		)
+	)
+	(text "V 1.1"
+		(exclude_from_sim no)
+		(at 272.034 193.548 0)
+		(effects
+			(font
+				(size 1.27 1.27)
+			)
 		)
 	)
