File: front_panel.kicad_sch (KiCad schematic)
At the start: 4 parts

Commit message: Updated versioning
Other:
- note added: "V 1.0"
Changed lines of the file:
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@@
+		)
+	)
+	(text "V 1.0"
+		(exclude_from_sim no)
+		(at 185.42 131.572 0)
+		(effects
+			(font
+				(size 1.27 1.27)
+			)
 		)
 	)
