File: VCA 1.kicad_sch (KiCad schematic)
At the start: 62 parts, among them J1 Eurorack 2x8hs, J15 IN 1x8s, J2 OUT 1x3s, J3 CV 1x9s, Q1 2N3904, Q2 2N3904, U1 TL074, U2 AS2164

Commit message: Updated versioning
Other:
- note added: "V 1.2"
- note removed: "V 1.1"
Changed lines of the file:
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@@
 		)
 	)
-	(text "V 1.1"
+	(text "V 1.2"
 		(exclude_from_sim no)
 		(at 394.462 280.162 0)

Commit message: Updated trim pot footprints
Parts:
- RV10, RV7, RV8, RV9: footprint Potentiometer_THT:Potentiometer_Bourns_3296W_Vertical -> Potentiometer_THT:Potentiometer_Bourns_3296X_Horizontal
Changed lines of the file:
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@@
 			)
 		)
-		(property "Footprint" "Potentiometer_THT:Potentiometer_Bourns_3296W_Vertical"
+		(property "Footprint" "Potentiometer_THT:Potentiometer_Bourns_3296X_Horizontal"
 			(at 72.39 208.28 0)
 			(hide yes)
@@
 			)
 		)
-		(property "Footprint" "Potentiometer_THT:Potentiometer_Bourns_3296W_Vertical"
+		(property "Footprint" "Potentiometer_THT:Potentiometer_Bourns_3296X_Horizontal"
 			(at 72.39 185.42 0)
 			(hide yes)
@@
 			)
 		)
-		(property "Footprint" "Potentiometer_THT:Potentiometer_Bourns_3296W_Vertical"
+		(property "Footprint" "Potentiometer_THT:Potentiometer_Bourns_3296X_Horizontal"
 			(at 73.66 60.96 0)
 			(hide yes)
@@
 			)
 		)
-		(property "Footprint" "Potentiometer_THT:Potentiometer_Bourns_3296W_Vertical"
+		(property "Footprint" "Potentiometer_THT:Potentiometer_Bourns_3296X_Horizontal"
 			(at 73.66 83.82 0)
 			(hide yes)

Commit message: Created custom AS2164 symbol, updated schematic, pcb and readme.
Parts:
- removed U2: AS2164, Package_DIP:DIP-16_W7.62mm, symbol Audio:SSI2164
- added D4, D5: LED, LED_THT:LED_D3.0mm_FlatTop, symbol Device:LED
- added H10, H11, H12, H9: (no value), MountingHole:MountingHole_3.2mm_M3, symbol Mechanical:MountingHole
- added H5, H6, H7, H8: (no value), MountingHole:MountingHole_2.7mm_M2.5, symbol Mechanical:MountingHole
- added J10: CV2, Connector_Audio:Jack_3.5mm_QingPu_WQP-PJ398SM_Vertical_CircularHoles, symbol Connector_Audio:AudioJack2_SwitchT
- added J11: IN2, Connector_Audio:Jack_3.5mm_QingPu_WQP-PJ398SM_Vertical_CircularHoles, symbol Connector_Audio:AudioJack2_SwitchT
- added J12: IN 1x8h, Connector_PinHeader_2.54mm:PinHeader_1x08_P2.54mm_Vertical, symbol Connector:Conn_01x08_Pin
- added J13: OUT1, Connector_Audio:Jack_3.5mm_QingPu_WQP-PJ398SM_Vertical_CircularHoles, symbol Connector_Audio:AudioJack2_SwitchT
- added J14: OUT2, Connector_Audio:Jack_3.5mm_QingPu_WQP-PJ398SM_Vertical_CircularHoles, symbol Connector_Audio:AudioJack2_SwitchT
- added J5: CV 1x9h, Connector_PinHeader_2.54mm:PinHeader_1x09_P2.54mm_Vertical, symbol Connector:Conn_01x09_Pin
- added J6: OUT 1x3h, Connector_PinHeader_2.54mm:PinHeader_1x03_P2.54mm_Vertical, symbol Connector:Conn_01x03_Pin
- added J8: CV1, Connector_Audio:Jack_3.5mm_QingPu_WQP-PJ398SM_Vertical_CircularHoles, symbol Connector_Audio:AudioJack2_SwitchT
- added J9: IN1, Connector_Audio:Jack_3.5mm_QingPu_WQP-PJ398SM_Vertical_CircularHoles, symbol Connector_Audio:AudioJack2_SwitchT
- added RV1, RV2, RV5, RV6: 10K B, Potentiometer_THT:Potentiometer_Alps_RK09L_Single_Vertical, symbol Device:R_Potentiometer
- added RV3, RV4: 50K B, Potentiometer_THT:Potentiometer_Alps_RK09L_Single_Vertical, symbol Device:R_Potentiometer
- added U2: AS2164, Package_DIP:DIP-16_W7.62mm, symbol AS2164:AS2164
Connections:
- net +12v: now also U2.16 (VCC)
- net -12v: now also C8.2, U2.9 (VEE); no longer C8.1
- net GND: now also C8.1, D4.1 (K), D5.1 (K), J10.S, J11.S, J13.S, J14.S, J6.3 (Pin_3), J8.S, J9.S, RV1.1, RV2.1, U2.8 (GND); no longer C8.2
- net at C11.1, R11.1, U1.12 (+): now also U2.4 (OUT)
- net at C9.2, J15.2 (Pin_2), U1.1: now also U2.3 (CV)
- net at C9.1, R4.2, R5.2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: now also U2.5 (OUT)
- net at R21.2: now also U2.1 (MODE)
- net at R17.2, R18.1: now also U2.10 (IN)
- net at C12.2, J15.6 (Pin_6), U1.7: now also U2.11 (CV)
- net at C14.1, R22.1, U1.9 (-): now also U2.12 (OUT)
- net at C12.1, R13.2, R14.2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: now also U2.13 (OUT)
- net at J15.7 (Pin_7): now also U2.14 (CV)
- net at R16.2: now also U2.15 (IN)
- net at R10.1, R9.2: now also U2.2 (IN)
- net at J15.3 (Pin_3): now also U2.6 (CV)
- net at R7.2: now also U2.7 (IN)
- new net: D4.2 (A), J5.1 (Pin_1)
- new net: J5.2 (Pin_2), J8.T, RV1.3
- new net: J5.3 (Pin_3), RV1.2
- new net: J5.4 (Pin_4), RV3.2
- new net: J5.5 (Pin_5), RV3.3, RV4.3
- new net: J5.6 (Pin_6), RV4.2
- new net: J5.7 (Pin_7), RV2.2
- new net: J10.T, J5.8 (Pin_8), RV2.3
- new net: D5.2 (A), J5.9 (Pin_9)
- new net: J14.T, J6.2 (Pin_2)
- new net: J12.8 (Pin_8), RV6.1
- new net: J12.7 (Pin_7), RV6.2
- new net: J12.6 (Pin_6), RV6.3
- new net: J11.T, J12.5 (Pin_5)
- new net: J13.T, J6.1 (Pin_1)
- new net: J12.1 (Pin_1), J9.T
- new net: J12.4 (Pin_4), RV5.1
- new net: J12.3 (Pin_3), RV5.2
- new net: J12.2 (Pin_2), RV5.3
- no-connect marks 6 -> 14
Other:
- removed sheet Controls
- removed sheet Front Panel
- note added: "Curve 1"
- note added: "Curve 2"
- note added: "Dual VCA I (main and control boards)"
- note added: "Level 1"
- note added: "Level 2"
- note added: "Main control and front panel drill holes"
- note added: "Offset 1"
- note added: "Offset 2"
- note added: "V 1.3"
- note removed: "Dual VCA I (main board)"
- note removed: "V 1.2"
- moved on the sheet: C10, C11, C12, C13, C14, C5, C6, C9, H1, H2, H3, H4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
